Commit message: adding TiaGo

File: fer_moveit/config/fer.ros2_control.xacro (robot description, xacro)
@@ -6,5 +6,5 @@
             <hardware>
                 <!-- By default, set up controllers for simulation. This won't work on real hardware -->
-                <plugin>mock_components/GenericSystem</plugin>
+                <plugin>gazebo_ros2_control/GazeboSystem</plugin>
             </hardware>
             <joint name="fer_joint1">
@@ -65,4 +65,9 @@
             </joint>
         </ros2_control>
+        <gazebo>
+            <plugin filename="libgazebo_ros2_control.so" name="gazebo_ros2_control">
+                <parameters>$(find fer_moveit)/config/ros2_controllers.yaml</parameters>
+            </plugin>
+        </gazebo>
     </xacro:macro>
 </robot>

File: fer_moveit/config/fer.urdf (robot description, URDF)
Before this commit: robot fer, 14 links, 13 joints
Links:
- link fer_hand: geometry collision mesh filename=package://franka_description/meshes/robot_ee/franka_hand_wh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; visual mesh filename=package://franka_description/meshes/robot_ee/franka_hand_wh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
- link fer_leftfinger: geometry collision box size=17.5e-3 15.2e-3 18.5e-3; collision box size=17.5e-3 7e-3 23.5e-3
- link fer_link0: geometry collision mesh filename=package://franka_description/meshes/robot_arms/fer/collisio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; visual mesh filename=package://franka_description/meshes/robot_arms/fer/visual/l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
- link fer_link1: geometry collision mesh filename=package://franka_description/meshes/robot_arms/fer/collisio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; visual mesh filename=package://franka_description/meshes/robot_arms/fer/visual/l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
- link fer_link2: geometry collision mesh filename=package://franka_description/meshes/robot_arms/fer/collisio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; visual mesh filename=package://franka_description/meshes/robot_arms/fer/visual/l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
- link fer_link3: geometry collision mesh filename=package://franka_description/meshes/robot_arms/fer/collisio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; visual mesh filename=package://franka_description/meshes/robot_arms/fer/visual/l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
- link fer_link4: geometry collision mesh filename=package://franka_description/meshes/robot_arms/fer/collisio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; visual mesh filename=package://franka_description/meshes/robot_arms/fer/visual/l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
- link fer_link5: geometry collision mesh filename=package://franka_description/meshes/robot_arms/fer/collisio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; visual mesh filename=package://franka_description/meshes/robot_arms/fer/visual/l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
- link fer_link6: geometry collision mesh filename=package://franka_description/meshes/robot_arms/fer/collisio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; visual mesh filename=package://franka_description/meshes/robot_arms/fer/visual/l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
- link fer_link7: geometry collision mesh filename=package://franka_description/meshes/robot_arms/fer/collisio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; visual mesh filename=package://franka_description/meshes/robot_arms/fer/visual/l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
- link fer_rightfinger: geometry collision box size=17.5e-3 15.2e-3 18.5e-3; collision box size=17.5e-3 7e-3 23.5e-3

Commit message: With docker file but packages are not portable yet

File: fer_moveit/config/fer.ros2_control.xacro (robot description, xacro)
@@ -3,71 +3,4 @@
     <xacro:macro name="fer_ros2_control" params="name initial_positions_file">
         <xacro:property name="initial_positions" value="${load_yaml(initial_positions_file)['initial_positions']}"/>
-        <ros2_control name="${name}" type="system">
-            <hardware>
-                <!-- By default, set up controllers for simulation. This won't work on real hardware -->
-                <plugin>gazebo_ros2_control/GazeboSystem</plugin>
-            </hardware>
-            <joint name="fer_joint1">
-                <command_interface name="position"/>
-                <state_interface name="position">
-                  <param name="initial_value">${initial_positions['fer_joint1']}</param>
-                </state_interface>
-                <state_interface name="velocity"/>
-            </joint>
-            <joint name="fer_joint2">
-                <command_interface name="position"/>
-                <state_interface name="position">
-                  <param name="initial_value">${initial_positions['fer_joint2']}</param>
-                </state_interface>
-                <state_interface name="velocity"/>
-            </joint>
-            <joint name="fer_joint3">
-                <command_interface name="position"/>
-                <state_interface name="position">
-                  <param name="initial_value">${initial_positions['fer_joint3']}</param>
-                </state_interface>
-                <state_interface name="velocity"/>
-            </joint>
-            <joint name="fer_joint4">
-                <command_interface name="position"/>
-                <state_interface name="position">
-                  <param name="initial_value">${initial_positions['fer_joint4']}</param>
-                </state_interface>
-                <state_interface name="velocity"/>
-            </joint>
-            <joint name="fer_joint5">
-                <command_interface name="position"/>
-                <state_interface name="position">
-                  <param name="initial_value">${initial_positions['fer_joint5']}</param>
-                </state_interface>
-                <state_interface name="velocity"/>
-            </joint>
-            <joint name="fer_joint6">
-                <command_interface name="position"/>
-                <state_interface name="position">
-                  <param name="initial_value">${initial_positions['fer_joint6']}</param>
-                </state_interface>
-                <state_interface name="velocity"/>
-            </joint>
-            <joint name="fer_joint7">
-                <command_interface name="position"/>
-                <state_interface name="position">
-                  <param name="initial_value">${initial_positions['fer_joint7']}</param>
-                </state_interface>
-                <state_interface name="velocity"/>
-            </joint>
-            <joint name="fer_finger_joint1">
-                <command_interface name="position"/>
-                <state_interface name="position">
-                  <param name="initial_value">${initial_positions['fer_finger_joint1']}</param>
-                </state_interface>
-                <state_interface name="velocity"/>
-            </joint>
-        </ros2_control>
-        <gazebo>
-            <plugin filename="libgazebo_ros2_control.so" name="gazebo_ros2_control">
-                <parameters>$(find fer_moveit)/config/ros2_controllers.yaml</parameters>
-            </plugin>
-        </gazebo>
     </xacro:macro>
 </robot>

File: fer_moveit/config/fer.urdf.xacro (robot description, xacro)
@@ -5,5 +5,6 @@
     <xacro:include filename="$(find franka_description)/robots/fer/fer.urdf.xacro" />
     <!-- Import control_xacro -->
-    <xacro:include filename="fer.ros2_control.xacro" />
-    <xacro:fer_ros2_control name="FakeSystem" initial_positions_file="$(arg initial_positions_file)"/>
+    <!--<xacro:include filename="fer.ros2_control.xacro" /> -->
+    <xacro:include filename="custom_fer.ros2_control.xacro" />
+    <xacro:custom_fer_ros2_control name="GazeboSystem" initial_positions_file="$(arg initial_positions_file)"/>
 </robot>
